File: KiCAD_Projektdateien/workshop_teil3/APC.kicad_pcb (KiCad board)
At the start: 2 copper layers, 94 x 57 mm, 20 parts, among them J1 Conn_01x02, SW1 SW_SPDT, U1 NE556

Commit message: Created fabrication files
Parts:
- added FID1: Fiducial, Fiducial:Fiducial_1mm_Mask2mm, F.Cu at (172.0, 54.0)
- added FID2: Fiducial, Fiducial:Fiducial_1mm_Mask2mm, F.Cu at (168.0, 96.0)
- added FID3: Fiducial, Fiducial:Fiducial_1mm_Mask2mm, F.Cu at (91.0, 54.0)
Other:
- board text added: "OFF"
- board text added: "ON"
Changed lines of the file:
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@@
   (general
     (thickness 1.6)
-    (drawings 5)
+    (drawings 7)
     (tracks 113)
     (zones 0)
-    (modules 20)
+    (modules 23)
     (nets 11)
   )
@@
       (outputformat 1)
       (mirror false)
-      (drillshape 1)
+      (drillshape 0)
       (scaleselection 1)
-      (outputdirectory ""))
+      (outputdirectory "./Fabrication/"))
   )
   (net 0 "")
@@
     (add_net GND)
     (add_net "Net-(BT1-Pad1)")
+  )
+  (module Fiducial:Fiducial_1mm_Mask2mm (layer F.Cu)
+    (at 91 54)
+    (descr "Circular Fiducial, 1mm bare copper, 2mm soldermask opening (Level A)")
+    (tags fiducial)
+    (attr smd)
+    (fp_text reference FID3 (at 0 -2) (layer F.SilkS) hide
+      (effects (font (size 1 1) (thickness 0.15)))
+    )
+    (fp_text value Fiducial (at 0 2) (layer F.Fab)
+      (effects (font (size 1 1) (thickness 0.15)))
+    )
+    (fp_circle (center 0 0) (end 1.25 0) (layer F.CrtYd) (width 0.05))
+    (fp_text user %R (at 0 0) (layer F.Fab)
+      (effects (font (size 0.4 0.4) (thickness 0.06)))
+    )
+    (fp_circle (center 0 0) (end 1 0) (layer F.Fab) (width 0.1))
+    (pad "" smd circle (at 0 0) (size 1 1) (layers F.Cu F.Mask)
+      (solder_mask_margin 0.5) (clearance 0.5))
+  )
+  (module Fiducial:Fiducial_1mm_Mask2mm (layer F.Cu)
+    (at 168 96)
+    (descr "Circular Fiducial, 1mm bare copper, 2mm soldermask opening (Level A)")
+    (tags fiducial)
+    (attr smd)
+    (fp_text reference FID2 (at 0 -2) (layer F.SilkS) hide
+      (effects (font (size 1 1) (thickness 0.15)))
+    )
+    (fp_text value Fiducial (at 0 2) (layer F.Fab)
+      (effects (font (size 1 1) (thickness 0.15)))
+    )
+    (fp_circle (center 0 0) (end 1.25 0) (layer F.CrtYd) (width 0.05))
+    (fp_text user %R (at 0 0) (layer F.Fab)
+      (effects (font (size 0.4 0.4) (thickness 0.06)))
+    )
+    (fp_circle (center 0 0) (end 1 0) (layer F.Fab) (width 0.1))
+    (pad "" smd circle (at 0 0) (size 1 1) (layers F.Cu F.Mask)
+      (solder_mask_margin 0.5) (clearance 0.5))
+  )
+  (module Fiducial:Fiducial_1mm_Mask2mm (layer F.Cu)
+    (at 172 54)
+    (descr "Circular Fiducial, 1mm bare copper, 2mm soldermask opening (Level A)")
+    (tags fiducial)
+    (attr smd)
+    (fp_text reference FID1 (at 0 -2) (layer F.SilkS) hide
+      (effects (font (size 1 1) (thickness 0.15)))
+    )
+    (fp_text value Fiducial (at 0 2) (layer F.Fab)
+      (effects (font (size 1 1) (thickness 0.15)))
+    )
+    (fp_circle (center 0 0) (end 1.25 0) (layer F.CrtYd) (width 0.05))
+    (fp_text user %R (at 0 0) (layer F.Fab)
+      (effects (font (size 0.4 0.4) (thickness 0.06)))
+    )
+    (fp_circle (center 0 0) (end 1 0) (layer F.Fab) (width 0.1))
+    (pad "" smd circle (at 0 0) (size 1 1) (layers F.Cu F.Mask)
+      (solder_mask_margin 0.5) (clearance 0.5))
   )
   (module Package_SO:SOIC-14_3.9x8.7mm_P1.27mm (layer F.Cu)
@@
     )
   )
+  (gr_text OFF (at 127.5 47 180) (layer F.SilkS)
+    (effects (font (size 1.5 1.5) (thickness 0.3)))
+  )
+  (gr_text ON (at 137 47 180) (layer F.SilkS)
+    (effects (font (size 1.5 1.5) (thickness 0.3)))
+  )
   (gr_text "Atari\nPunk\nConsole\nV0.1" (at 135.5 89) (layer F.SilkS)
